File: pcb/ttrpg9000.kicad_sch (KiCad schematic)
At the start: 53 parts, among them J1 AVR-ISP-6, J2 C1x6, J3 C1x6, SW1 SW_SPDT, SW2 RotaryEncoder_Switch, SW3 RotaryEncoder_Switch, U1 ATtiny4313-S, U2 LP2950-3.3_TO252

Commit message: Remove LED circuits and 3.3V regulator
Parts:
- removed C2: 2.2u, Resistor_SMD:R_1206_3216Metric_Pad1.30x1.75mm_HandSolder, symbol Device:C
- removed D1: RED, LED_SMD:LED_0805_2012Metric_Pad1.15x1.40mm_HandSolder, symbol Device:LED
- removed D2: GRN, LED_SMD:LED_0805_2012Metric_Pad1.15x1.40mm_HandSolder, symbol Device:LED
- removed D3: BLU, LED_SMD:LED_0805_2012Metric_Pad1.15x1.40mm_HandSolder, symbol Device:LED
- removed R12, R13: 100R, Resistor_SMD:R_0805_2012Metric_Pad1.20x1.40mm_HandSolder, symbol Device:R
- removed R14: 10R, Resistor_SMD:R_0805_2012Metric_Pad1.20x1.40mm_HandSolder, symbol Device:R
- removed R15, R16, R17: 1.2R, Resistor_SMD:R_0805_2012Metric_Pad1.20x1.40mm_HandSolder, symbol Device:R
- removed U2: LP2950-3.3_TO252, Project:TO-252-2_HandSolder, symbol Regulator_Linear:LP2950-3.3_TO252
- BT1: value 2x3V -> 3V
Connections:
- net +6V is gone; now on net +3V0: BT1.1 (+), C1.1
- net +3V3 renamed +3V0
- net +3V3_2 renamed +3V0_2
- net +3V0_2: no longer DS1.1 (A1+), DS1.2 (A2+), DS1.3 (A3+)
- no-connect marks 2 -> 11
Other:
- note added: "Battery and power switch"
- note added: "NOTE: +3V0/+3V0_2 and GND/GND_2 connected via ribbon cable"
- note removed: "NOTE: +3V3/+3V3_2 and GND/GND_2 connected via ribbon cable"
- note removed: "Power regulator"
- moved on the sheet: C1, C11, C12, C14, C7, C8, C9

Commit message: Replace battery holder with single cell available from JLCPCB
Parts:
- BT1: footprint Project:Keystone_3025-2 -> Project:BAT_AAA-BAT-054-P06
Changed lines of the file:
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@@
 			)
 		)
-		(property "Footprint" "Project:Keystone_3025-2"
+		(property "Footprint" "Project:BAT_AAA-BAT-054-P06"
 			(at 50.8 168.656 90)
 			(effects

Commit message: Change battery mounting hole radius
Parts:
- C1: LCSC Part # (none) -> C1848
Changed lines of the file:
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@@
+			)
+		)
+		(property "LCSC Part #" "C1848"
+			(at 59.69 158.75 90)
+			(effects
+				(font
+					(size 1.27 1.27)
+				)
+				(hide yes)
 			)
 		)
